File: PCB/protoCtrl/protoCtrl.sch (EAGLE design)
At the start: 122 parts, among them IC1 AVR_XMEGA_A1_100A, U1 MCP73831, U2 V_REG_LDOSMD, U3 FT232RLSSOP, U4 ADG726BSUZ, U5 SD_CARD_SOCKET4UCON, U6 AD9283BRSZ-80REAL, U7 AD9283BRSZ-80REAL

Commit message: adding images and cleaning up
Other:
- note added: "BOARD INTERCONNECT"
- note added: "TFT LCD"
- moved on the sheet: C14, C16, C17, C18, C19, C6, CN1, H1, H2, H3, IC1, JP3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
